File: KICad_Files/KICad_Files.kicad_sch (KiCad schematic)
At the start: 48 parts, among them J1 Conn_01x03_Pin, J10 Conn_01x03_MountingPin, J2 Conn_01x03_Pin, J3 Conn_01x06, J4 Conn_01x06, J5 Conn_01x03_Pin, J6 Conn_01x02_Pin, J7 USB_C_Receptacle_USB2.0_14P, J8 Conn_01x03_MountingPin, J9 Conn_01x03_MountingPin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

Commit message: Changed from 3 to 2 connector because of ESP32-C3 Limitations
Parts:
- removed J8: Conn_01x03_MountingPin, Connector_Molex:Molex_PicoBlade_53047-0310_1x03_P1.25mm_Vertical, symbol Connector_Generic:Conn_01x03
- J7: value USB_C_Receptacle_USB2.0_14P -> USB_C_Receptacle_USB2.0_16P
Connections:
- net LED3 renamed Boot
Changed lines of the file:
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@@
 	)
 	(junction
-		(at 360.68 196.85)
-		(diameter 0)
-		(color 0 0 0 0)
-	)
-	(junction
 		(at 157.48 177.8)
 		(diameter 0)
@@
 	)
 	(junction
-		(at 358.14 184.15)
-		(diameter 0)
-		(color 0 0 0 0)
-	)
-	(junction
 		(at 148.59 96.52)
 		(diameter 0)
@@
 	(wire
 		(pts
-			(xy 360.68 186.69) (xy 360.68 196.85)
-		)
-		(stroke
-			(width 0)
-			(type default)
-		)
-	)
-	(wire
-		(pts
 			(xy 365.76 35.56) (xy 365.76 44.45)
 		)
@@
 	(wire
 		(pts
-			(xy 358.14 184.15) (xy 358.14 194.31)
-		)
-		(stroke
-			(width 0)
-			(type default)
-		)
-	)
-	(wire
-		(pts
 			(xy 334.01 148.59) (xy 341.63 148.59)
 		)
@@
 	(wire
 		(pts
+			(xy 358.14 187.96) (xy 358.14 194.31)
+		)
+		(stroke
+			(width 0)
+			(type default)
+		)
+	)
+	(wire
+		(pts
 			(xy 349.25 44.45) (xy 349.25 35.56)
 		)
@@
 	(wire
 		(pts
-			(xy 355.6 181.61) (xy 365.76 181.61)
-		)
-		(stroke
-			(width 0)
-			(type default)
-		)
-	)
-	(wire
-		(pts
 			(xy 246.38 175.26) (xy 248.92 175.26)
 		)
@@
 	(wire
 		(pts
-			(xy 360.68 186.69) (xy 365.76 186.69)
-		)
-		(stroke
-			(width 0)
-			(type default)
-		)
-	)
-	(wire
-		(pts
 			(xy 185.42 135.89) (xy 185.42 143.51)
 		)
@@
 	(wire
 		(pts
-			(xy 358.14 179.07) (xy 358.14 184.15)
-		)
-		(stroke
-			(width 0)
-			(type default)
-		)
-	)
-	(wire
-		(pts
 			(xy 342.9 113.03) (xy 339.09 113.03)
 		)
@@
 	(wire
 		(pts
-			(xy 358.14 184.15) (xy 365.76 184.15)
-		)
-		(stroke
-			(width 0)
-			(type default)
-		)
-	)
-	(wire
-		(pts
 			(xy 217.17 95.25) (xy 217.17 100.33)
 		)
@@
 	)
 	(rectangle
-		(start 341.63 172.72)
+		(start 341.63 180.34)
 		(end 398.78 215.9)
 		(stroke
@@
 	(text "connector to LEDs"
 		(exclude_from_sim no)
-		(at 341.63 170.942 0)
+		(at 341.63 179.324 0)
 		(effects
 			(font
@@
 		)
 	)
-	(label "LED3"
+	(label "Boot"
 		(at 233.68 160.02 180)
 		(effects
@@
 		)
 	)
-	(label "LED3"
+	(label "Boot"
 		(at 372.11 78.74 180)
 		(effects
@@
 		)
 	)
-	(label "LED3"
-		(at 355.6 181.61 180)
-		(effects
-			(font
-				(size 1.27 1.27)
-			)
-			(justify right bottom)
-		)
-	)
 	(label "XTAL_P"
 		(at 208.28 105.41 180)
@@
 	(symbol
 		(lib_id "power:+5V")
-		(at 358.14 179.07 0)
+		(at 358.14 187.96 0)
 		(unit 1)
 		(exclude_from_sim no)
@@
 		(fields_autoplaced yes)
 		(property "Reference" "#PWR27"
-			(at 358.14 182.88 0)
+			(at 358.14 191.77 0)
 			(effects
 				(font
@@
 		)
 		(property "Value" "+5V"
-			(at 358.14 173.99 0)
+			(at 358.14 182.88 0)
 			(effects
 				(font
@@
 		)
 		(property "Footprint" ""
-			(at 358.14 179.07 0)
+			(at 358.14 187.96 0)
 			(effects
 				(font
@@
 		)
 		(property "Datasheet" ""
-			(at 358.14 179.07 0)
+			(at 358.14 187.96 0)
 			(effects
 				(font
@@
 		)
 		(property "Description" "Power symbol creates a global label with name \"+5V\""
-			(at 358.14 179.07 0)
+			(at 358.14 187.96 0)
 			(effects
 				(font
@@
 		(dnp no)
 		(property "Reference" "J7"
-			(at 384.81 119.3799 90)
+			(at 387.985 120.65 0)
 			(effects
 				(font
 					(size 1.27 1.27)
 				)
-				(justify left)
 			)
 		)
-		(property "Value" "USB_C_Receptacle_USB2.0_14P"
-			(at 350.774 108.458 90)
+		(property "Value" "USB_C_Receptacle_USB2.0_16P"
+			(at 385.445 120.65 0)
 			(effects
 				(font
 					(size 1.27 1.27)
 				)
-				(justify left)
 			)
 		)
@@
 					(unit 1)
 				)
-			)
-		)
-	)
-	(symbol
-		(lib_id "Connector_Generic:Conn_01x03")
-		(at 370.84 184.15 0)
-		(unit 1)
-		(exclude_from_sim no)
-		(in_bom yes)
-		(on_board yes)
-		(dnp no)
-		(fields_autoplaced yes)
-		(property "Reference" "J8"
-			(at 373.38 182.8799 0)
-			(effects
-				(font
-					(size 1.27 1.27)
-				)
-				(justify left)
-			)
-		)
-		(property "Value" "Conn_01x03_MountingPin"
-			(at 373.38 185.4199 0)
-			(effects
-				(font
-					(size 1.27 1.27)
-				)
-				(justify left)
-			)
-		)
-		(property "Footprint" "Connector_Molex:Molex_PicoBlade_53047-0310_1x03_P1.25mm_Vertical"
-			(at 370.84 184.15 0)
-			(effects
-				(font
-					(size 1.27 1.27)
-				)
-				(hide yes)
-			)
-		)
-		(property "Datasheet" "~"
-			(at 370.84 184.15 0)
-			(effects
-				(font
-					(size 1.27 1.27)
-				)
-				(hide yes)
-			)
-		)
-		(property "Description" "Generic connector, single row, 01x03, script generated (kicad-library-utils/schlib/autogen/connector/)"
-			(at 370.84 184.15 0)
-			(effects
-				(font
-					(size 1.27 1.27)
-				)
-				(hide yes)
-			)
-		)
-		(pin "3"
-		)
-		(pin "2"
-		)
-		(pin "1"
-		)
-		(instances
-			(project ""
-				(path "/34061aa1-1595-4a0a-9524-9b9b15681d54"
-					(reference "J8")
-					(unit 1)
-				)

Commit message: Switched the pi-filter components to 0402 size and changed the values
Parts:
- C3, C4: value 3p3 -> 1p2; footprint Capacitor_SMD:C_0603_1608Metric_Pad1.08x0.95mm_HandSolder -> Capacitor_SMD:C_0402_1005Metric_Pad0.74x0.62mm_HandSolder
- L1: value 2n2 -> 3n9; footprint Inductor_SMD:L_0603_1608Metric -> Inductor_SMD:L_0402_1005Metric_Pad0.77x0.64mm_HandSolder
Changed lines of the file:
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@@
 			)
 		)
-		(property "Value" "3p3"
+		(property "Value" "1p2"
 			(at 138.43 104.14 0)
 			(effects
@@
 			)
 		)
-		(property "Footprint" "Capacitor_SMD:C_0603_1608Metric_Pad1.08x0.95mm_HandSolder"
+		(property "Footprint" "Capacitor_SMD:C_0402_1005Metric_Pad0.74x0.62mm_HandSolder"
 			(at 136.8552 106.68 0)
 			(effects
@@
 			)
 		)
-		(property "Value" "3p3"
+		(property "Value" "1p2"
 			(at 151.13 104.14 0)
 			(effects
@@
 			)
 		)
-		(property "Footprint" "Capacitor_SMD:C_0603_1608Metric_Pad1.08x0.95mm_HandSolder"
+		(property "Footprint" "Capacitor_SMD:C_0402_1005Metric_Pad0.74x0.62mm_HandSolder"
 			(at 149.5552 106.68 0)
 			(effects
@@
 			)
 		)
-		(property "Value" "2n2"
+		(property "Value" "3n9"
 			(at 142.24 93.98 90)
 			(effects
@@
 			)
 		)
-		(property "Footprint" "Inductor_SMD:L_0603_1608Metric"
+		(property "Footprint" "Inductor_SMD:L_0402_1005Metric_Pad0.77x0.64mm_HandSolder"
 			(at 134.62 87.63 90)
 			(effects
@@
 					(size 1.27 1.27)
 				)
-				(hide yes)
 			)
 		)

Commit message: Switched crystal size and changed GPIO02 to be pulled high instead of low
Parts:
- Y1: footprint Crystal:Crystal_SMD_3225-4Pin_3.2x2.5mm -> Crystal:Crystal_SMD_1210-4Pin_1.2x1.0mm
Connections:
- net +3.3V: now also R6.1
- net GND: no longer R6.1
Changed lines of the file:
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@@
 	(wire
 		(pts
-			(xy 236.22 144.78) (xy 236.22 152.4)
-		)
-		(stroke
-			(width 0)
-			(type default)
-		)
-	)
-	(wire
-		(pts
 			(xy 320.04 55.88) (xy 307.34 55.88)
 		)
@@
 	(wire
 		(pts
+			(xy 219.71 152.4) (xy 219.71 148.59)
+		)
+		(stroke
+			(width 0)
+			(type default)
+		)
+	)
+	(wire
+		(pts
 			(xy 266.7 143.51) (xy 271.78 143.51)
 		)
@@
 	(wire
 		(pts
-			(xy 231.14 144.78) (xy 236.22 144.78)
-		)
-		(stroke
-			(width 0)
-			(type default)
-		)
-	)
-	(wire
-		(pts
 			(xy 142.24 106.68) (xy 142.24 110.49)
 		)
@@
 	(wire
 		(pts
-			(xy 231.14 144.78) (xy 231.14 146.05)
-		)
-		(stroke
-			(width 0)
-			(type default)
-		)
-	)
-	(wire
-		(pts
 			(xy 308.61 27.94) (xy 306.07 27.94)
 		)
@@
 	(wire
 		(pts
+			(xy 219.71 152.4) (xy 238.76 152.4)
+		)
+		(stroke
+			(width 0)
+			(type default)
+		)
+	)
+	(wire
+		(pts
 			(xy 217.17 95.25) (xy 217.17 100.33)
 		)
@@
 	(wire
 		(pts
-			(xy 236.22 152.4) (xy 238.76 152.4)
-		)
-		(stroke
-			(width 0)
-			(type default)
-		)
-	)
-	(wire
-		(pts
 			(xy 387.35 29.21) (xy 389.89 29.21)
 		)
@@
 	(symbol
 		(lib_id "power:GND")
-		(at 231.14 146.05 0)
-		(unit 1)
-		(exclude_from_sim no)
-		(in_bom yes)
-		(on_board yes)
-		(dnp no)
-		(fields_autoplaced yes)
-		(property "Reference" "#PWR20"
-			(at 231.14 152.4 0)
-			(effects
-				(font
-					(size 1.27 1.27)
-				)
-				(hide yes)
-			)
-		)
-		(property "Value" "GND"
-			(at 231.14 151.13 0)
-			(effects
-				(font
-					(size 1.27 1.27)
-				)
-			)
-		)
-		(property "Footprint" ""
-			(at 231.14 146.05 0)
-			(effects
-				(font
-					(size 1.27 1.27)
-				)
-				(hide yes)
-			)
-		)
-		(property "Datasheet" ""
-			(at 231.14 146.05 0)
-			(effects
-				(font
-					(size 1.27 1.27)
-				)
-				(hide yes)
-			)
-		)
-		(property "Description" "Power symbol creates a global label with name \"GND\" , ground"
-			(at 231.14 146.05 0)
-			(effects
-				(font
-					(size 1.27 1.27)
-				)
-				(hide yes)
-			)
-		)
-		(pin "1"
-		)
-		(instances
-			(project "KICad_Files"
-				(path "/34061aa1-1595-4a0a-9524-9b9b15681d54"
-					(reference "#PWR20")
-					(unit 1)
-				)
-			)
-		)
-	)
-	(symbol
-		(lib_id "power:GND")
 		(at 285.75 120.65 0)
 		(unit 1)
@@
 	)
 	(symbol
+		(lib_id "power:+3.3V")
+		(at 219.71 148.59 0)
+		(mirror y)
+		(unit 1)
+		(exclude_from_sim no)
+		(in_bom yes)
+		(on_board yes)
+		(dnp no)
+		(property "Reference" "#PWR20"
+			(at 219.71 152.4 0)
+			(effects
+				(font
+					(size 1.27 1.27)
+				)
+				(hide yes)
+			)
+		)
+		(property "Value" "+3.3V"
+			(at 219.71 143.51 0)
+			(effects
+				(font
+					(size 1.27 1.27)
+				)
+			)
+		)
+		(property "Footprint" ""
+			(at 219.71 148.59 0)
+			(effects
+				(font
+					(size 1.27 1.27)
+				)
+				(hide yes)
+			)
+		)
+		(property "Datasheet" ""
+			(at 219.71 148.59 0)
+			(effects
+				(font
+					(size 1.27 1.27)
+				)
+				(hide yes)
+			)
+		)
+		(property "Description" "Power symbol creates a global label with name \"+3.3V\""
+			(at 219.71 148.59 0)
+			(effects
+				(font
+					(size 1.27 1.27)
+				)
+				(hide yes)
+			)
+		)
+		(pin "1"
+		)
+		(instances
+			(project "KICad_Files"
+				(path "/34061aa1-1595-4a0a-9524-9b9b15681d54"
+					(reference "#PWR20")
+					(unit 1)
+				)
+			)
+		)
+	)
+	(symbol
 		(lib_id "power:GND")
 		(at 179.07 161.29 0)
@@
 			)
 		)
-		(property "Footprint" "Crystal:Crystal_SMD_3225-4Pin_3.2x2.5mm"
+		(property "Footprint" "Crystal:Crystal_SMD_1210-4Pin_1.2x1.0mm"
 			(at 217.17 105.41 0)
 			(effects
